File: 03 - Hadware/05 - Kicad/DC_DC_CONVERTER/DC_DC_CONVERTER.kicad_sch (KiCad schematic)
At the start: 0 parts

Commit message: Schematic final version 04.05.25
Parts:
- added C10, C14, C7, C8, C9: 22pF, Capacitor_THT:CP_Radial_D8.0mm_P5.00mm, symbol Device:C
- added C11, C5: 100nF, Capacitor_THT:CP_Radial_D8.0mm_P5.00mm, symbol Device:C
- added C12: 100uF, Capacitor_THT:CP_Radial_D8.0mm_P5.00mm, symbol Device:C
- added C13: 1000uF, Capacitor_THT:CP_Radial_D8.0mm_P5.00mm, symbol Device:C
- added C16, C17: 135uF, Capacitor_THT:CP_Radial_D8.0mm_P5.00mm, symbol Device:C
- added C18, C19: 47uF, Capacitor_THT:CP_Radial_D8.0mm_P5.00mm, symbol Device:C
- added C3: 10uF, Capacitor_THT:CP_Radial_D8.0mm_P5.00mm, symbol Device:C
- added C4: 22uF, Capacitor_THT:CP_Radial_D5.0mm_P2.50mm, symbol Device:C
- added C6: C_Polarized 10uF, Capacitor_THT:CP_Radial_D8.0mm_P5.00mm, symbol Device:C_Polarized
- added D1, D2, D3: LED, LED_THT:LED_D3.0mm, symbol Device:LED
- added D18, D19: 1N5338BG, Library:DIOAD1543W101L863D368, symbol 1N5338B:1N5338BG
- added D22, D23, D4, D5, D6, D7: 1N4004, Diode_THT:D_DO-41_SOD81_P10.16mm_Horizontal, symbol Diode:1N4004
- added D8: 1N5822, Diode_THT:D_DO-201AD_P15.24mm_Horizontal, symbol Diode:1N5822
- added J2: USB_B, USBR-B-S-S-O-TH:USB_B_OST_USB-B1HSxx_Horizontal, symbol Connector:USB_B
- added J3, J4: Screw_Terminal_01x02, Library:HANDSON_KF301-2P, symbol Connector:Screw_Terminal_01x02
- added JP1: Jumper_3_Open, Library:SAMTEC_MTSW-101-06-T-T-100, symbol Jumper:Jumper_3_Open
- added K1, K2, K3, K4: SRD-05VDC-SL-C, Library:RELAY_SRD-05VDC-SL-C, symbol SRD-05VDC-SL-C:SRD-05VDC-SL-C
- added L1: 100uH, Inductor_THT:L_Radial_D12.0mm_P6.00mm_Murata_1900R, symbol Device:L
- added L2: 2.78mH, Inductor_THT:L_Radial_D12.0mm_P6.00mm_Murata_1900R, symbol Device:L
- added Q1, Q3, Q5, Q7: BC547, Package_TO_SOT_THT:TO-92_Inline, symbol Transistor_BJT:BC547
- added Q10, Q2, Q27, Q28, Q32, Q33, Q34, Q35, Q36, Q4, Q6: IRLZ44N, Package_TO_SOT_THT:TO-220-3_Vertical, symbol Transistor_FET:IRLZ44N
- added R1: 0.25, Resistor_THT:R_Axial_DIN0414_L11.9mm_D4.5mm_P15.24mm_Horizontal, symbol Device:R
- added R10, R12, R13, R15, R16, R48, R49, R50, R51, R9: 220, Resistor_THT:R_Axial_DIN0414_L11.9mm_D4.5mm_P15.24mm_Horizontal, symbol Device:R
- added R11, R14, R40, R42: 10K, Resistor_THT:R_Axial_DIN0414_L11.9mm_D4.5mm_P15.24mm_Horizontal, symbol Device:R
- added R2: 3.15, Resistor_THT:R_Axial_DIN0414_L11.9mm_D4.5mm_P15.24mm_Horizontal, symbol Device:R
- added R3, R4, R5, R6, R7: 1K, Resistor_THT:R_Axial_DIN0414_L11.9mm_D4.5mm_P15.24mm_Horizontal, symbol Device:R
- added R39, R41: 100K, Resistor_THT:R_Axial_DIN0414_L11.9mm_D4.5mm_P15.24mm_Horizontal, symbol Device:R
- added R47: 47, Resistor_THT:R_Axial_DIN0414_L11.9mm_D4.5mm_P15.24mm_Horizontal, symbol Device:R
- added R8: 1M, Resistor_THT:R_Axial_DIN0414_L11.9mm_D4.5mm_P15.24mm_Horizontal, symbol Device:R
- added U2: LT1083-ADJ, ul_LT1083CP-PBF:TO-3P_P_LIT, symbol Regulator_Linear:LT1083-ADJ
- added U3: ATmega328P-P, Package_DIP:DIP-28_W7.62mm, symbol MCU_Microchip_ATmega:ATmega328P-P
- added U4: CH340G, Package_SO:SOIC-16_3.9x9.9mm_P1.27mm, symbol Interface_USB:CH340G
- added U5: LCD-16X2, LCD-16X2:MODULE_LCD-16X2, symbol LCD-16x2:LCD-16X2
- added U6: LM2576HVT-5.0, T05A_TEX, symbol LM2576HVT-5.0:LM2576HVT-5.0
- added U8, U9: IR2104, Library:DIP762W45P254L988H533Q8, symbol Driver_FET:IR2104
- added Y1: 16MHz, Crystal:Crystal_HC49-4H_Vertical, symbol Device:Crystal
- added Y2: 12MHz, Crystal:Crystal_HC49-4H_Vertical, symbol Device:Crystal
Connections:
- new net: R1.2, R2.1, U2.1 (ADJ)
- new net: Q33.1 (G), R48.1
- new net: R48.2, U8.7 (HO)
- new net: D4.2 (A), K1.A2, Q1.1 (C)
- new net: K1.NC, Q2.2 (D), R11.2
- new net: R49.2, U8.5 (LO)
- new net: C18.1, D22.1 (K), U8.8 (VB)
- new net: L2.1, Q10.2 (D), Q6.3 (S)
- new net: Q34.1 (G), R49.1
- new net: Q7.2 (B), R16.1
- new net: D3.2 (A), R7.2
- new net: L2.2, Q27.3 (S), Q28.2 (D)
- new net: D1.2 (A), R3.2
- new net: C9.1, R8.2, U3.10 (XTAL2/PB7), Y1.2
- new net: C10.1, R8.1, U3.9 (XTAL1/PB6), Y1.1
- new net: D8.1 (K), L1.1, U6.2 (OUT)
- new net: R5.1, U4.3 (RXD)
- new net: Q2.1 (G), R10.1
- new net: Q4.1 (G), R13.1
- new net: K2.NC, Q4.2 (D), R14.2
- new net: D2.2 (A), R6.2
- new net: Q1.2 (B), R9.1
- new net: D7.2 (A), K4.A2, Q7.1 (C)
- new net: C19.1, D23.1 (K), U9.8 (VB)
- new net: Q35.1 (G), R50.1
- new net: R50.2, U9.7 (HO)
- new net: D5.2 (A), K2.A2, Q3.1 (C)
- new net: Q3.2 (B), R12.1
- new net: Q36.1 (G), R51.1
- new net: R51.2, U9.5 (LO)
- new net: D6.2 (A), K3.A2, Q5.1 (C)
- new net: Q5.2 (B), R15.1
- new net: C14.1, U4.13 (~{DTR})
- new net: R4.1, U4.2 (TXD)
- new net: C7.1, U4.7 (XI), Y2.1
- new net: C8.1, U4.8 (XO), Y2.2
- new net 1-D: C19.2, Q32.2 (D), Q35.3 (S), Q36.2 (D), R47.2, U9.6 (VS)
- new net 17V: C4.1, D22.2 (A), D23.2 (A), Q33.2 (D), Q35.2 (D), R1.1, R11.1, R14.1, R47.1, U2.2 (VO), U8.1 (VCC), U8.3 (~{SD}), U9.1 (VCC), U9.3 (~{SD})
- new net 3.3V_Output: U4.4 (V3)
- new net 5V: C11.1, C13.1, D4.1 (K), D5.1 (K), D6.1 (K), D7.1 (K), K1.A1, K2.A1, K3.A1, K4.A1, L1.2, R6.1, R7.1, U3.20 (AVCC), U3.7 (VCC), U5.15 (A), U5.2 (VDD), U5.3 (VO), U6.4 (FB)
- new net 5V_USB: C5.1, C6.1, J2.1 (VBUS), R3.1, U4.16 (VCC)
- new net A_Side: C16.1, J3.2 (Pin_2), JP1.1 (A), Q6.2 (D), R41.1
- new net A_Side_ADC: D19.1, R41.2, R42.1, U3.23 (PC0)
- new net B_Side: C17.1, J4.1 (Pin_1), JP1.3 (B), Q27.2 (D), R39.1
- new net B_Side_ADC: D18.1, R39.2, R40.1, U3.24 (PC1)
- new net Control_R1A: R9.2, U3.4 (PD2)
- new net Control_R1B: R10.2, U3.5 (PD3)
- new net Control_R2A: R15.2, U3.25 (PC2)
- new net Control_R3A: R12.2, U3.26 (PC3)
- new net Control_R3B: R13.2, U3.27 (PC4)
- new net Control_R4A: R16.2, U3.28 (PC5)
- new net D: C18.2, K1.NO, K2.NO, K3.NO, K4.NO, Q32.1 (G), Q33.3 (S), Q34.2 (D), U8.6 (VS)
- new net D4: U3.13 (PD7), U5.11 (DB4)
- new net D5: U3.12 (PD6), U5.12 (DB5)
- new net D6: U3.11 (PD5), U5.13 (DB6)
- new net D7: U3.6 (PD4), U5.14 (DB7)
- new net DATA_PIN_1: J2.3 (D+), U4.5 (UD+)
- new net DATA_PIN_2: J2.2 (D-), U4.6 (UD-)
- new net E: U3.17 (PB3), U5.6 (E)
- new net GND: C10.2, C11.2, C12.2, C13.2, C16.2, C17.2, C3.2, C4.2, C9.2, D18.2, D19.2, D8.2 (A), J3.1 (Pin_1), J4.2 (Pin_2), K3.NC, K4.NC, Q1.3 (E), Q10.3 (S), Q2.3 (S), Q28.3 (S), Q3.3 (E), Q32.3 (S), Q34.3 (S), Q36.3 (S), Q4.3 (S), Q5.3 (E), Q7.3 (E), R2.2, R40.2, R42.2, U3.22 (GND), U3.8 (GND), U5.1 (VSS), U5.10 (DB3), U5.16 (K), U5.5 (R/W), U5.7 (DB0), U5.8 (DB1), U5.9 (DB2), U6.3 (GND), U6.5 (*ON/OFF), U8.4 (COM), U9.4 (COM)
- new net GND1: C5.2, C6.2, C7.2, C8.2, D1.1 (K), J2.4 (GND), J2.5 (Shield), U4.1 (GND)
- new net POWER: C12.1, C3.1, JP1.2 (C), U2.3 (VI), U6.1 (VIN)
- new net R1_OUTPUT: K1.COM, Q6.1 (G)
- new net R2_OUTPUT: K3.COM, Q10.1 (G)
- new net R3_OUTPUT: K2.COM, Q27.1 (G)
- new net R4_OUTPUT: K4.COM, Q28.1 (G)
- new net RESET_USB: C14.2, U3.1 (~{RESET}/PC6)
- new net RS: U3.18 (PB4), U5.4 (RS)
- new net RX: D3.1 (K), R5.2, U3.3 (PD1)
- new net SWITCH_1: U3.15 (PB1), U8.2 (IN)
- new net SWITCH_2: U3.16 (PB2), U9.2 (IN)
- new net TX: D2.1 (K), R4.2, U3.2 (PD0)
- no-connect marks 0 -> 9
Other:
- note added: "17V Regulator"
- note added: "5V Regulator"
- note added: "DISPLAY LCD - DEBUG/MONITORING"
- note added: "Final Year Project By Electronic Engineering - IFSP (Federal Institute of São Paulo)"
- note added: "GATE DRIVERS"
- note added: "MCU"
- note added: "POWER SUPPLIER Vi - Voltage Input (18V ~ 30V) Vi - Voltage Output(7 ~ 55)"
- note added: "RELAY_1"
- note added: "RELAY_2"
- note added: "RELAY_3"
- note added: "RELAY_4"
- note added: "SWITCHERS"
- note added: "Tantalum"
- note added: "USB"
- note added: "USB/SERIAL CONVERSOR"
- note added: "VOLTAGE SELECTION SIDE"
- note added: "Voltage Monitoring"
- note added: "Vout- V adj = 1.25V IR1 = 5A (worst Case) R1 = 1.25/5A = 0.25 Ohms -> 6.25W (High Power) Vr = (Vout - 1.25) = (17V - 1.25V) = 15.75V R2 = V/I = 15.75/5A = 3.15 Ohms -> 78.75W (high Power)."
- note added: "Worst Case Voltage = 55V Vout = Vin* (R2(R1+R2)) Vin = 55V Vout = 5V R1 = 100K, R2 = 10K"
- note removed: "Final Year Project By Electronic Engineering - IFSP (Institute Federal of São Paulo)"
- title: (none) -> BIDIRECTIONAL DC DC CONVERTER

Commit message: release pires 18.05.25 update: Schematic/Layout/Priteus simulation/Matlab Simulation/Monogroph
Parts:
- JP1: footprint Library:SAMTEC_MTSW-101-06-T-T-100 -> Connector_PinHeader_2.54mm:PinHeader_1x03_P2.54mm_Vertical
Changed lines of the file:
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@@
 			)
 		)
-		(property "Footprint" "Library:SAMTEC_MTSW-101-06-T-T-100"
+		(property "Footprint" "Connector_PinHeader_2.54mm:PinHeader_1x03_P2.54mm_Vertical"
 			(at 57.15 36.83 0)
 			(effects
@@
 			)
 		)
-		(property "Datasheet" " ~"
+		(property "Datasheet" "~"
 			(at 228.6 48.26 0)
 			(effects
@@
 			)
 		)
-		(property "Description" "\n                        \n                            Display Development Tools 16x2 Black on Green Char LCD w Backlight\n                        \n"
+		(property "Description" "Display Development Tools 16x2 Black on Green Char LCD w Backlight"
 			(at 59.69 163.83 0)
 			(effects

Commit message: add picture folder
Parts:
- removed Q2, Q4: IRLZ44N, Package_TO_SOT_THT:TO-220-3_Vertical, symbol Transistor_FET:IRLZ44N
- removed R10, R13: 220, Resistor_THT:R_Axial_DIN0414_L11.9mm_D4.5mm_P15.24mm_Horizontal, symbol Device:R
Connections:
- net Control_R1B: no longer names the net of U3.5 (PD3)
- net Control_R3B: no longer names the net of U3.27 (PC4)
- no-connect marks 9 -> 11
Other:
- moved on the sheet: R11
